Commit message: add all links and joints to urdf. add stl files for collision

File: src/description/urdf/description.urdf.xacro (robot description, xacro)
@@ -27,6 +27,82 @@
         </visual>
         <collision>
+            <origin rpy="-${PI/2} 0 0" xyz="0 0 0"/>
             <geometry>
-                <cylinder length="0.6" radius="0.2"/>
+                <mesh filename="${path}/base_collision.stl" scale="${scale}"/>
+            </geometry>
+        </collision>
+    </link>
+    <link name="rotary_link">
+        <xacro:default_inertial mass="0.05"/>
+        <visual>
+            <origin rpy="-${PI/2} 0 -${PI/2}" xyz="0 0 0"/>
+            <geometry>
+                <mesh filename="${path}/rotary.stl" scale="${scale}"/>
+            </geometry>
+        </visual>
+        <collision>
+            <origin rpy="-${PI/2} 0 -${PI/2}" xyz="0 0 0"/>
+            <geometry>
+                <mesh filename="${path}/rotary_collision.stl" scale="${scale}"/>
+            </geometry>
+        </collision>
+    </link>
+    <link name="arm_1_link">
+        <xacro:default_inertial mass="0.1"/>
+        <visual>
+            <origin rpy="0 ${PI/2} ${PI}" xyz="0 0 0"/>
+            <geometry>
+                <mesh filename="${path}/arm_1.stl" scale="${scale}"/>
+            </geometry>
+        </visual>
+        <collision>
+            <origin rpy="0 ${PI/2} ${PI}" xyz="0 0 0"/>
+            <geometry>
+                <mesh filename="${path}/arm_1_collision.stl" scale="${scale}"/>
+            </geometry>
+        </collision>
+    </link>
+    <link name="arm_2_link">
+        <xacro:default_inertial mass="0.1"/>
+        <visual>
+            <origin rpy="0 ${PI/2} 0" xyz="0 0 0"/>
+            <geometry>
+                <mesh filename="${path}/arm_2.stl" scale="${scale}"/>
+            </geometry>
+        </visual>
+        <collision>
+            <origin rpy="0 ${PI/2} 0" xyz="0 0 0"/>
+            <geometry>
+                <mesh filename="${path}/arm_2_collision.stl" scale="${scale}"/>
+            </geometry>
+        </collision>
+    </link>
+    <link name="arm_3_link">
+        <xacro:default_inertial mass="0.1"/>
+        <visual>
+            <origin rpy="0 ${PI/2} ${PI}" xyz="0 0 0"/>
+            <geometry>
+                <mesh filename="${path}/arm_3.stl" scale="${scale}"/>
+            </geometry>
+        </visual>
+        <collision>
+            <origin rpy="0 ${PI/2} ${PI}" xyz="0 0 0"/>
+            <geometry>
+                <mesh filename="${path}/arm_3_collision.stl" scale="${scale}"/>
+            </geometry>
+        </collision>
+    </link>
+    <link name="gripper_link">
+        <xacro:default_inertial mass="0.05"/>
+        <visual>
+            <origin rpy="-${PI/2} 0 ${PI}" xyz="0 0 0"/>
+            <geometry>
+                <mesh filename="${path}/gripper_3.stl" scale="${scale}"/>
+            </geometry>
+        </visual>
+        <collision>
+            <origin rpy="-${PI/2} 0 ${PI}" xyz="0 0 0"/>
+            <geometry>
+                <mesh filename="${path}/gripper_3_collision.stl" scale="${scale}"/>
             </geometry>
         </collision>
@@ -38,3 +114,43 @@
         <origin xyz="0 0 0" rpy="0 0 0"/>
     </joint>
+    <joint name ="joint_1" type="revolute">
+        <parent link="base_link"/>
+        <child link = "rotary_link"/>
+        <origin xyz="0 0 1.3"/>
+        <axis xyz="0 0 1"/>
+        <limit lower="-${PI / 2}" upper="${PI / 2}"
+               effort="${effort}" velocity="${velocity}"/>
+    </joint>
+    <joint name ="joint_2" type="revolute">
+        <parent link="rotary_link"/>
+        <child link = "arm_1_link"/>
+        <origin xyz="0 0 0"/>
+        <axis xyz="1 0 0"/>
+        <limit lower="-${PI / 2}" upper="${PI / 2}"
+               effort="${effort}" velocity="${velocity}"/>
+    </joint>
+    <joint name ="joint_3" type="revolute">
+        <parent link="arm_1_link"/>
+        <child link = "arm_2_link"/>
+        <origin xyz="0 0 1.545"/>
+        <axis xyz="1 0 0"/>
+        <limit lower="-${PI / 2}" upper="${PI / 2}"
+               effort="${effort}" velocity="${velocity}"/>
+    </joint>
+    <joint name ="joint_4" type="revolute">
+        <parent link="arm_2_link"/>
+        <child link = "arm_3_link"/>
+        <origin xyz="0 0 1.945"/>
+        <axis xyz="1 0 0"/>
+        <limit lower="-${PI / 2}" upper="${PI / 2}"
+               effort="${effort}" velocity="${velocity}"/>
+    </joint>
+    <joint name ="joint_5" type="revolute">
+        <parent link="arm_3_link"/>
+        <child link = "gripper_link"/>
+        <origin xyz="0 0 0.88"/>
+        <axis xyz="0 0 1"/>
+        <limit lower="-${PI / 2}" upper="${PI / 2}"
+               effort="${effort}" velocity="${velocity}"/>
+    </joint>
 </robot>

Commit message: add controller

File: src/description/urdf/description.urdf.xacro (robot description, xacro)
@@ -11,7 +11,5 @@
             <origin xyz="0 0 0" rpy="0 0 0"/>
             <mass value="${mass}" />
-            <inertia ixx="1.0" ixy="0.0" ixz="0.0"
-                        iyy="1.0" iyz="0.0"
-                        izz="1.0" />
+            <inertia ixx="1.0" ixy="0.0" ixz="0.0" iyy="1.0" iyz="0.0" izz="1.0" />
         </inertial>
     </xacro:macro>
@@ -154,3 +152,11 @@
                effort="${effort}" velocity="${velocity}"/>
     </joint>
+    <!-- Control -->
+    <xacro:include filename="$(find description)/urdf/control.xacro" />
+    <!-- Gazebo (for Humble)-->
+    <gazebo>
+        <plugin filename="ign_ros2_control-system" name="ign_ros2_control::IgnitionROS2ControlPlugin">
+            <parameters>$(find controller)/config/controller.yaml</parameters>
+        </plugin>
+    </gazebo>
 </robot>

Commit message: add virtual joint for tip

File: src/description/urdf/description.urdf.xacro (robot description, xacro)
@@ -106,4 +106,5 @@
         </collision>
     </link>
+    <link name="tip"/>
     <!-- JOINTS -->
     <joint name="virtual_joint" type="fixed">
@@ -152,4 +153,9 @@
                effort="${effort}" velocity="${velocity}"/>
     </joint>
+    <joint name="virtual_joint_tip" type="fixed">
+        <parent link="gripper_link"/>
+        <child link="tip"/>
+        <origin xyz="0 0 1.56" rpy="0 0 0"/>
+    </joint>
     <!-- Gazebo (for Humble)-->
     <gazebo>

Commit message: update firmware command to handle negatives. update urdfs.

File: src/description/urdf/description.urdf.xacro (robot description, xacro)
@@ -20,5 +20,5 @@
         <xacro:default_inertial mass="0.2"/>
         <visual>
-            <origin rpy="-${PI/2} 0 0" xyz="0 0 0"/>
+            <origin rpy="0 0 0" xyz="0 0 0"/>
             <geometry>
                 <mesh filename="${path}/base.stl" scale="${scale}"/>
@@ -26,5 +26,5 @@
         </visual>
         <collision>
-            <origin rpy="-${PI/2} 0 0" xyz="0 0 0"/>
+            <origin rpy="0 0 0" xyz="0 0 0"/>
             <geometry>
                 <mesh filename="${path}/base_collision.stl" scale="${scale}"/>
@@ -35,5 +35,5 @@
         <xacro:default_inertial mass="0.05"/>
         <visual>
-            <origin rpy="-${PI/2} 0 -${PI/2}" xyz="0 0 0"/>
+            <origin rpy="0 0 ${PI/2}" xyz="0 0 0"/>
             <geometry>
                 <mesh filename="${path}/rotary.stl" scale="${scale}"/>

Commit message: modify to match latest mechanics. define better home position

File: src/description/urdf/description.urdf.xacro (robot description, xacro)
@@ -117,5 +117,5 @@
         <parent link="base_link"/>
         <child link = "rotary_link"/>
-        <origin xyz="0 0 1.3"/>
+        <origin xyz="0 0 1.47"/>
         <axis xyz="0 0 1"/>
         <limit lower="-${PI / 2}" upper="${PI / 2}"
@@ -157,5 +157,5 @@
         <parent link="gripper_link"/>
         <child link="tip"/>
-        <origin xyz="0 0 1.56" rpy="0 0 0"/>
+        <origin xyz="0 0 1.75" rpy="0 0 0"/>
     </joint>
     <!-- Gazebo (for Humble)-->
