Commit message: Add temporary joint_6 for 6-DOF simulation
A massless wrist_link and a Y-axis joint_6 make the arm 6-DOF in simulation only: no servo or mesh behind it, and the real joint will replace it. Kinematics at joint_6 = 0 are unchanged, so recorded poses still hold, and Pilz blending works again. The gripper moved to joint_7; the hardware path is deliberately left broken.

File: src/description/urdf/control.xacro (robot description, xacro)
@@ -51,4 +51,11 @@
             <state_interface name="position"/>
         </joint>
+        <joint name="joint_6">
+            <command_interface name="position">
+            <param name="min">-${PI / 2}</param>
+            <param name="max">${PI / 2}</param>
+            </command_interface>
+            <state_interface name="position"/>
+        </joint>
     </ros2_control>
 </robot>

File: src/description/urdf/description.urdf.xacro (robot description, xacro)
@@ -92,4 +92,11 @@
         </collision>
     </link>
+    <!-- TEMPORARY, SIMULATION ONLY. Placeholder for the sixth DOF: carries no mesh
+         of its own, so at joint_6 = 0 the robot looks exactly as it did when the
+         arm had 5 joints. The real joint, with its own geometry and a servo behind
+         it, will replace this. See "The sixth joint" in CLAUDE.md. -->
+    <link name="wrist_link">
+        <xacro:default_inertial mass="0.01"/>
+    </link>
     <link name="gripper_link">
         <xacro:default_inertial mass="0.05"/>
@@ -148,7 +155,15 @@
     <joint name ="joint_5" type="revolute">
         <parent link="arm_3_link"/>
-        <child link = "gripper_link"/>
+        <child link = "wrist_link"/>
         <origin xyz="0 0 0.88"/>
         <axis xyz="0 0 1"/>
+        <limit lower="-${PI / 2}" upper="${PI / 2}"
+               effort="${effort}" velocity="${velocity}"/>
+    </joint>
+    <joint name ="joint_6" type="revolute">
+        <parent link="wrist_link"/>
+        <child link = "gripper_link"/>
+        <origin xyz="0 0 0"/>
+        <axis xyz="0 1 0"/>
         <limit lower="-${PI / 2}" upper="${PI / 2}"
                effort="${effort}" velocity="${velocity}"/>
